File: Hardware/Reflow Oven.kicad_sch (KiCad schematic)
At the start: 11 parts, among them J1 SW, J2 ENC, J3 SENS_AMP_1, J4 SENS_AMP_2, J6 2350513-2, J7 2350513-2, J8 2350513-3

Commit message: minor work left on rev1
Parts:
- removed J3: SENS_AMP_1, symbol Connector_Generic:Conn_01x08
- removed J4: SENS_AMP_2, symbol Connector_Generic:Conn_01x08
- added C22, C23, C24: 10n, symbol Device:C_Small
- added J10: 2350513-2, KiCAD Library:2350513-2, symbol Connector_Generic:Conn_01x02
- added J3, J4, J5: Adafruit 4101, Connector_PinHeader_2.54mm:PinHeader_1x09_P2.54mm_Vertical, symbol Connector_Generic:Conn_01x09
- added J6: GC9A01 1.28" TFT, Connector_PinHeader_2.54mm:PinHeader_1x07_P2.54mm_Vertical, symbol Connector_Generic:Conn_01x07
- added P1: ~, Cuprum:IRM015, symbol Cuprum:IRM-01-05
- added R1: 2k2, Cuprum:R_0603_1608Metric, symbol Device:R_Small
- H1, H2, H3, H4: footprint (none) -> MountingHole:MountingHole_3.2mm_M3_DIN965_Pad
- J1: footprint (none) -> Connector_PinHeader_2.54mm:PinHeader_1x04_P2.54mm_Vertical
- J2: footprint (none) -> Connector_PinHeader_2.54mm:PinHeader_1x05_P2.54mm_Vertical
- J7: renamed from J8; footprint (none) -> KiCAD Library:2350513-3
- J8: renamed from J6; footprint (none) -> KiCAD Library:2350513-2
- J9: renamed from J7; footprint (none) -> KiCAD Library:2350513-2
Connections:
- net NEUT is gone; now on net Earth: J7.1 (Pin_1)
- net +3V3: now also J3.1 (Pin_1), J4.1 (Pin_1), J5.1 (Pin_1), J6.1 (Pin_1)
- net ALARM1A: now also J3.5 (Pin_5)
- net ALARM1B: now also J4.5 (Pin_5)
- net ALARM2A: now also J3.6 (Pin_6)
- net ALARM2B: now also J4.6 (Pin_6)
- net ALARM3A: now also J3.7 (Pin_7)
- net ALARM3B: now also J4.7 (Pin_7)
- net ALARM4A: now also J3.8 (Pin_8)
- net ALARM4B: now also J4.8 (Pin_8)
- net Button Filter/SW_OUT: no longer J1.2 (Pin_2)
- net GND: now also C24.1, J3.2 (Pin_2), J4.2 (Pin_2), J5.2 (Pin_2), J5.9 (Pin_9), J6.2 (Pin_2), P1.2 (V-), R1.1
- net LCD_CS: now also J6.6 (Pin_6)
- net LCD_D/C: now also J6.5 (Pin_5)
- net LCD_MOSI: now also J6.4 (Pin_4)
- net LCD_RST: now also J6.7 (Pin_7)
- net LCD_SCK: now also J6.3 (Pin_3)
- net SCL: now also J3.3 (Pin_3), J4.3 (Pin_3), J5.3 (Pin_3)
- net SDA: now also J3.4 (Pin_4), J4.4 (Pin_4), J5.4 (Pin_4)
- net ENC_Filter/ENC_A_IN renamed ENC_A
- net ENC_Filter/ENC_B_IN renamed ENC_B
- net ENC_Filter/ENC_SW_IN renamed ENC_SW
- net Earth_Protective renamed Earth
- net Earth: now also C22.2, C23.2, C24.2; no longer J7.3 (Pin_3)
- net LINE renamed Live
- net Live: now also C23.1, P1.4 (L)
- net Microcontroller/SW_LED renamed Microcontroller Alarm/SW_LED
- new net: J4.9 (Pin_9), R1.2
- new net +5V: P1.1 (V+)
- new net ALARM1C: J5.5 (Pin_5)
- new net ALARM2C: J5.6 (Pin_6)
- new net ALARM3C: J5.7 (Pin_7)
- new net ALARM4C: J5.8 (Pin_8)
- new net MOSFETs/SSR_3: J10.2 (Pin_2)
- new net MOSFETs/SSR_3_COM: J10.1 (Pin_1)
- new net Neutral: C22.1, J7.3 (Pin_3), P1.3 (N)
- new net SW: J1.2 (Pin_2)
- no-connect marks 0 -> 1
Other:
- removed sheet Display
- removed sheet Microcontroller
- removed sheet PawPad
- added sheet Microcontroller Alarm (Sheets/MicrocontrollerAlarm.kicad_sch)
- sheet MOSFETs ports: added MOSFET_3, SSR_3, SSR_3_COM; removed none
- note added: "I2C ADDR: 0x60"
- note added: "I2C ADDR: 0x61"
- note added: "I2C ADDR: 0x67"
- note added: "NOT PRESENT ON REV 1"
- note added: "Y-Capacitors"
- moved on the sheet: H1, H2, H3, H4, J1, J2, J7
