File: Hardware/Reflow Oven.kicad_pcb (KiCad board)
At the start: 4 copper layers, 100 x 50 mm, 84 parts, among them IC1 MCP1792T, J1 SW, J10 2350513-2, J11 USB4110-GF-A_REVB, J12 POW_SEL, J13 PawPad_SWD, J2 ENC, J3 Adafruit 4101, J4 Adafruit 4101, J5 Adafruit 4101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

Commit message: minor tweaks
Parts:
- moved C12 1.38 mm to (134.7, 96.8)
- moved G*** 1.15 mm to (187.8, 101.5)
Connections:
- J11 pad S1: GND -> unconnected-(J11-SHIELD-PadS1)
Routing:
- net +5V: track 6.95 -> 77.7 mm, vias 0 -> 3
- net VBUS: track 0.00 -> 34.9 mm, vias 0 -> 2
- net GND: track 46.4 -> 58.8 mm, vias 30 -> 38
- net Earth: track 0.00 -> 9.48 mm
- net +3V3: track 40.0 -> 45.1 mm, vias 9 -> 16
- added copper zone on F.Cu, net /ENC_A
- added copper zone on F.Cu, net /ENC_B
- added copper zone on F.Cu, net /ENC_SW
