File: Hardware/Sheets/Button Filter.kicad_sch (KiCad schematic)
At the start: 4 parts

Commit message: minor work left on rev1
Parts:
- removed JP1: Bypass Filter, symbol Jumper:SolderJumper_2_Open
- C19: footprint (none) -> KiCAD Library:C_0603_1608Metric
- R10, R9: footprint (none) -> Cuprum:R_0603_1608Metric
Changed lines of the file:
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@@
   (junction (at 121.92 90.17) (diameter 0) (color 0 0 0 0)
-  )
-  (junction (at 151.13 90.17) (diameter 0) (color 0 0 0 0)
-  )
-  (junction (at 134.62 90.17) (diameter 0) (color 0 0 0 0)
   )
   (junction (at 119.38 90.17) (diameter 0) (color 0 0 0 0)
@@
     (stroke (width 0) (type default))
   )
-  (wire (pts (xy 146.05 77.47) (xy 151.13 77.47))
-    (stroke (width 0) (type default))
-  )
-  (wire (pts (xy 151.13 77.47) (xy 151.13 90.17))
-    (stroke (width 0) (type default))
-  )
-  (wire (pts (xy 134.62 90.17) (xy 139.7 90.17))
-    (stroke (width 0) (type default))
-  )
-  (wire (pts (xy 138.43 77.47) (xy 134.62 77.47))
-    (stroke (width 0) (type default))
-  )
-  (wire (pts (xy 121.92 90.17) (xy 134.62 90.17))
+  (wire (pts (xy 121.92 90.17) (xy 139.7 90.17))
     (stroke (width 0) (type default))
   )
@@
     (stroke (width 0) (type default))
   )
-  (wire (pts (xy 134.62 77.47) (xy 134.62 90.17))
-    (stroke (width 0) (type default))
-  )
-  (wire (pts (xy 151.13 90.17) (xy 168.91 90.17))
+  (wire (pts (xy 144.78 90.17) (xy 168.91 90.17))
     (stroke (width 0) (type default))
   )
   (wire (pts (xy 113.03 90.17) (xy 119.38 90.17))
-    (stroke (width 0) (type default))
-  )
-  (wire (pts (xy 144.78 90.17) (xy 151.13 90.17))
     (stroke (width 0) (type default))
   )
@@
           (reference "#PWR017") (unit 1)
         )
-        (path "/a8f55c7f-bff8-431d-a8db-3e7e1d4b6c05/c8b8f2ff-0b9b-4830-841d-05219ecaf535"
-          (reference "#PWR012") (unit 1)
-        )
         (path "/a8f55c7f-bff8-431d-a8db-3e7e1d4b6c05/286b9674-44a4-4e8c-a366-fdc5002831c4"
           (reference "#PWR024") (unit 1)
         )
         (path "/a8f55c7f-bff8-431d-a8db-3e7e1d4b6c05/d70fecd1-5c35-4fe2-97e2-8d1a0a4635fd"
-          (reference "#PWR030") (unit 1)
+          (reference "#PWR021") (unit 1)
         )
       )
@@
     )
   )
-  (symbol (lib_id "Jumper:SolderJumper_2_Open") (at 142.24 77.47 0) (unit 1)
-    (in_bom yes) (on_board yes) (dnp no)
-    (property "Reference" "JP1" (at 142.24 74.93 0)
-      (effects (font (size 1.27 1.27)))
-    )
-    (property "Value" "Bypass Filter" (at 142.24 80.01 0)
-      (effects (font (size 1.27 1.27)))
-    )
-    (property "Footprint" "" (at 142.24 77.47 0)
-      (effects (font (size 1.27 1.27)) hide)
-    )
-    (property "Datasheet" "~" (at 142.24 77.47 0)
-      (effects (font (size 1.27 1.27)) hide)
-    )
-    (pin "1")
-    (pin "2")
-    (instances
-      (project "Reflow Oven"
-        (path "/a8f55c7f-bff8-431d-a8db-3e7e1d4b6c05"
-          (reference "JP1") (unit 1)
-        )
-        (path "/a8f55c7f-bff8-431d-a8db-3e7e1d4b6c05/286b9674-44a4-4e8c-a366-fdc5002831c4"
-          (reference "JP3") (unit 1)
-        )
-        (path "/a8f55c7f-bff8-431d-a8db-3e7e1d4b6c05/d70fecd1-5c35-4fe2-97e2-8d1a0a4635fd"
-          (reference "JP4") (unit 1)
-        )
-      )
-    )
-  )
   (symbol (lib_id "Device:C_Small") (at 121.92 95.25 0) (unit 1)
     (in_bom yes) (on_board yes) (dnp no) (fields_autoplaced)
@@
       (effects (font (size 1.27 1.27)) (justify left))
     )
-    (property "Footprint" "" (at 121.92 95.25 0)
+    (property "Footprint" "KiCAD Library:C_0603_1608Metric" (at 121.92 95.25 0)
       (effects (font (size 1.27 1.27)) hide)
     )
@@
         )
         (path "/a8f55c7f-bff8-431d-a8db-3e7e1d4b6c05/d70fecd1-5c35-4fe2-97e2-8d1a0a4635fd"
-          (reference "C20") (unit 1)
+          (reference "C4") (unit 1)
         )
       )
@@
       (effects (font (size 1.27 1.27)) (justify left))
     )
-    (property "Footprint" "" (at 119.38 85.09 0)
+    (property "Footprint" "Cuprum:R_0603_1608Metric" (at 119.38 85.09 0)
       (effects (font (size 1.27 1.27)) hide)
     )
@@
         )
         (path "/a8f55c7f-bff8-431d-a8db-3e7e1d4b6c05/d70fecd1-5c35-4fe2-97e2-8d1a0a4635fd"
-          (reference "R10") (unit 1)
+          (reference "R8") (unit 1)
         )
       )
@@
           (reference "#PWR018") (unit 1)
         )
-        (path "/a8f55c7f-bff8-431d-a8db-3e7e1d4b6c05/c8b8f2ff-0b9b-4830-841d-05219ecaf535"
-          (reference "#PWR013") (unit 1)
-        )
         (path "/a8f55c7f-bff8-431d-a8db-3e7e1d4b6c05/286b9674-44a4-4e8c-a366-fdc5002831c4"
           (reference "#PWR023") (unit 1)
         )
         (path "/a8f55c7f-bff8-431d-a8db-3e7e1d4b6c05/d70fecd1-5c35-4fe2-97e2-8d1a0a4635fd"
-          (reference "#PWR029") (unit 1)
+          (reference "#PWR020") (unit 1)
         )
       )
@@
       (effects (font (size 1.27 1.27)))
     )
-    (property "Footprint" "" (at 142.24 90.17 0)
+    (property "Footprint" "Cuprum:R_0603_1608Metric" (at 142.24 90.17 0)
       (effects (font (size 1.27 1.27)) hide)
     )
@@
         )
         (path "/a8f55c7f-bff8-431d-a8db-3e7e1d4b6c05/d70fecd1-5c35-4fe2-97e2-8d1a0a4635fd"
-          (reference "R11") (unit 1)
+          (reference "R9") (unit 1)
         )
       )
