File: Hardware/Sheets/Display.kicad_sch (KiCad schematic)
At the start: 7 parts, among them Q1 BC817

Commit message: minor work left on rev1
Parts:
- renumbered C21 to C22, C22 to C23, R12 to R14, R13 to R15, R14 to R16
Changed lines of the file:
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@@
   (symbol (lib_id "power:+3V3") (at 99.06 54.61 0) (unit 1)
     (in_bom yes) (on_board yes) (dnp no)
-    (property "Reference" "#PWR031" (at 99.06 58.42 0)
+    (property "Reference" "#PWR039" (at 99.06 58.42 0)
       (effects (font (size 1.27 1.27)) hide)
     )
@@
       (project "Reflow Oven"
         (path "/a8f55c7f-bff8-431d-a8db-3e7e1d4b6c05/a3b6b84f-45d1-47f7-925b-5d1aaeec6fa2"
-          (reference "#PWR031") (unit 1)
+          (reference "#PWR039") (unit 1)
         )
       )
@@
   (symbol (lib_id "power:GND") (at 164.465 95.25 0) (unit 1)
     (in_bom yes) (on_board yes) (dnp no) (fields_autoplaced)
-    (property "Reference" "#PWR035" (at 164.465 101.6 0)
+    (property "Reference" "#PWR043" (at 164.465 101.6 0)
       (effects (font (size 1.27 1.27)) hide)
     )
@@
       (project "Reflow Oven"
         (path "/a8f55c7f-bff8-431d-a8db-3e7e1d4b6c05/a3b6b84f-45d1-47f7-925b-5d1aaeec6fa2"
-          (reference "#PWR035") (unit 1)
+          (reference "#PWR043") (unit 1)
         )
       )
@@
   (symbol (lib_id "Device:R_Small") (at 99.06 62.23 180) (unit 1)
     (in_bom yes) (on_board yes) (dnp no) (fields_autoplaced)
-    (property "Reference" "R13" (at 101.6 60.9599 0)
+    (property "Reference" "R15" (at 101.6 60.9599 0)
       (effects (font (size 1.27 1.27)) (justify right))
     )
@@
       (project "Reflow Oven"
         (path "/a8f55c7f-bff8-431d-a8db-3e7e1d4b6c05/a3b6b84f-45d1-47f7-925b-5d1aaeec6fa2"
-          (reference "R13") (unit 1)
+          (reference "R15") (unit 1)
         )
       )
@@
   (symbol (lib_id "power:GND") (at 109.22 76.835 0) (unit 1)
     (in_bom yes) (on_board yes) (dnp no)
-    (property "Reference" "#PWR034" (at 109.22 83.185 0)
+    (property "Reference" "#PWR042" (at 109.22 83.185 0)
       (effects (font (size 1.27 1.27)) hide)
     )
@@
       (project "Reflow Oven"
         (path "/a8f55c7f-bff8-431d-a8db-3e7e1d4b6c05/a3b6b84f-45d1-47f7-925b-5d1aaeec6fa2"
-          (reference "#PWR034") (unit 1)
+          (reference "#PWR042") (unit 1)
         )
       )
@@
   (symbol (lib_id "Device:C_Small") (at 107.95 109.22 0) (unit 1)
     (in_bom yes) (on_board yes) (dnp no)
-    (property "Reference" "C22" (at 110.2741 108.3178 0)
+    (property "Reference" "C23" (at 110.2741 108.3178 0)
       (effects (font (size 1.27 1.27)) (justify left))
     )
@@
       (project "Reflow Oven"
         (path "/a8f55c7f-bff8-431d-a8db-3e7e1d4b6c05/a3b6b84f-45d1-47f7-925b-5d1aaeec6fa2"
-          (reference "C22") (unit 1)
+          (reference "C23") (unit 1)
         )
       )
@@
   (symbol (lib_id "power:GND") (at 172.085 123.19 0) (unit 1)
     (in_bom yes) (on_board yes) (dnp no) (fields_autoplaced)
-    (property "Reference" "#PWR036" (at 172.085 129.54 0)
+    (property "Reference" "#PWR044" (at 172.085 129.54 0)
       (effects (font (size 1.27 1.27)) hide)
     )
@@
       (project "Reflow Oven"
         (path "/a8f55c7f-bff8-431d-a8db-3e7e1d4b6c05/a3b6b84f-45d1-47f7-925b-5d1aaeec6fa2"
-          (reference "#PWR036") (unit 1)
+          (reference "#PWR044") (unit 1)
         )
       )
@@
   (symbol (lib_id "Device:R_Small") (at 91.44 71.12 90) (unit 1)
     (in_bom yes) (on_board yes) (dnp no)
-    (property "Reference" "R12" (at 91.44 67.31 90)
+    (property "Reference" "R14" (at 91.44 67.31 90)
       (effects (font (size 1.27 1.27)))
     )
@@
       (project "Reflow Oven"
         (path "/a8f55c7f-bff8-431d-a8db-3e7e1d4b6c05/a3b6b84f-45d1-47f7-925b-5d1aaeec6fa2"
-          (reference "R12") (unit 1)
+          (reference "R14") (unit 1)
         )
       )
@@
   (symbol (lib_id "Device:C_Small") (at 99.06 109.22 0) (unit 1)
     (in_bom yes) (on_board yes) (dnp no)
-    (property "Reference" "C21" (at 101.3841 108.3178 0)
+    (property "Reference" "C22" (at 101.3841 108.3178 0)
       (effects (font (size 1.27 1.27)) (justify left))
     )
@@
       (project "Reflow Oven"
         (path "/a8f55c7f-bff8-431d-a8db-3e7e1d4b6c05/a3b6b84f-45d1-47f7-925b-5d1aaeec6fa2"
-          (reference "C21") (unit 1)
+          (reference "C22") (unit 1)
         )
       )
@@
   (symbol (lib_id "power:GND") (at 99.06 118.11 0) (unit 1)
     (in_bom yes) (on_board yes) (dnp no) (fields_autoplaced)
-    (property "Reference" "#PWR033" (at 99.06 124.46 0)
+    (property "Reference" "#PWR041" (at 99.06 124.46 0)
       (effects (font (size 1.27 1.27)) hide)
     )
@@
       (project "Reflow Oven"
         (path "/a8f55c7f-bff8-431d-a8db-3e7e1d4b6c05/a3b6b84f-45d1-47f7-925b-5d1aaeec6fa2"
-          (reference "#PWR033") (unit 1)
+          (reference "#PWR041") (unit 1)
         )
       )
@@
   (symbol (lib_id "power:+3V3") (at 99.06 100.33 0) (unit 1)
     (in_bom yes) (on_board yes) (dnp no) (fields_autoplaced)
-    (property "Reference" "#PWR032" (at 99.06 104.14 0)
+    (property "Reference" "#PWR040" (at 99.06 104.14 0)
       (effects (font (size 1.27 1.27)) hide)
     )
@@
       (project "Reflow Oven"
         (path "/a8f55c7f-bff8-431d-a8db-3e7e1d4b6c05/a3b6b84f-45d1-47f7-925b-5d1aaeec6fa2"
-          (reference "#PWR032") (unit 1)
+          (reference "#PWR040") (unit 1)
         )
       )
@@
   (symbol (lib_id "power:+3V3") (at 176.53 100.33 0) (unit 1)
     (in_bom yes) (on_board yes) (dnp no) (fields_autoplaced)
-    (property "Reference" "#PWR037" (at 176.53 104.14 0)
+    (property "Reference" "#PWR045" (at 176.53 104.14 0)
       (effects (font (size 1.27 1.27)) hide)
     )
@@
       (project "Reflow Oven"
         (path "/a8f55c7f-bff8-431d-a8db-3e7e1d4b6c05/a3b6b84f-45d1-47f7-925b-5d1aaeec6fa2"
-          (reference "#PWR037") (unit 1)
+          (reference "#PWR045") (unit 1)
         )
       )
@@
   (symbol (lib_id "Device:R_Small") (at 121.92 63.5 270) (unit 1)
     (in_bom yes) (on_board yes) (dnp no) (fields_autoplaced)
-    (property "Reference" "R14" (at 121.92 58.42 90)
+    (property "Reference" "R16" (at 121.92 58.42 90)
       (effects (font (size 1.27 1.27)))
     )
@@
       (project "Reflow Oven"
         (path "/a8f55c7f-bff8-431d-a8db-3e7e1d4b6c05/a3b6b84f-45d1-47f7-925b-5d1aaeec6fa2"
-          (reference "R14") (unit 1)
-        )
-      )
+          (reference "R16") (unit 1)
+        )
+      )
