File: Hardware/Sheets/ENC_Filter.kicad_sch (KiCad schematic)
At the start: 12 parts

Commit message: minor work left on rev1
Parts:
- removed JP1 (x3): Bypass Filter, symbol Jumper:SolderJumper_2_Open
- C1: renamed from C17; footprint (none) -> KiCAD Library:C_0603_1608Metric
- C2: renamed from C18; footprint (none) -> KiCAD Library:C_0603_1608Metric
- C3: renamed from C19; footprint (none) -> KiCAD Library:C_0603_1608Metric
- R2: renamed from R4; footprint (none) -> Cuprum:R_0603_1608Metric
- R3: renamed from R5; footprint (none) -> Cuprum:R_0603_1608Metric
- R4: renamed from R6; footprint (none) -> Cuprum:R_0603_1608Metric
- R5: renamed from R7; footprint (none) -> Cuprum:R_0603_1608Metric
- R6: renamed from R8; footprint (none) -> Cuprum:R_0603_1608Metric
- R7: renamed from R9; footprint (none) -> Cuprum:R_0603_1608Metric
Other:
- moved on the sheet: C1, C3, R2, R4, R5, R7
