File: Hardware/Sheets/MOSFETs.kicad_sch (KiCad schematic)
At the start: 8 parts, among them Q2 NMOS, Q3 NMOS

Commit message: minor work left on rev1
Parts:
- added D1, D2, D3: Red, Diode_SMD:D_0805_2012Metric, symbol Device:LED_Small
- added F3: Fuse, Fuse:Fuse_1206_3216Metric, symbol Device:Fuse
- added Q3: IRLML2060, Package_TO_SOT_SMD:SOT-23, symbol Simulation_SPICE:NMOS
- added R12, R15, R18: 270, Cuprum:R_0603_1608Metric, symbol Device:R_Small
- added R19: 100, Cuprum:R_0603_1608Metric, symbol Device:R_Small
- added R20: 10k, Cuprum:R_0603_1608Metric, symbol Device:R_Small
- F1, F2: footprint (none) -> Fuse:Fuse_1206_3216Metric
- Q1: renamed from Q2; value NMOS -> IRLML2060; footprint (none) -> Package_TO_SOT_SMD:SOT-23
- Q2: renamed from Q3; value NMOS -> IRLML2060; footprint (none) -> Package_TO_SOT_SMD:SOT-23
- R13: renamed from R18; footprint (none) -> Cuprum:R_0603_1608Metric
- R14: renamed from R17; footprint (none) -> Cuprum:R_0603_1608Metric
- R16: renamed from R20; footprint (none) -> Cuprum:R_0603_1608Metric
- R17: renamed from R19; footprint (none) -> Cuprum:R_0603_1608Metric
Connections:
- net GND: now also D1.1 (K), D2.1 (K), D3.1 (K), Q3.3 (S), R20.2
- net MOSFET_1: now also R12.1; no longer R14.1
- net MOSFET_2: now also R15.1; no longer R17.1
- net at Q1.2 (G), R13.2: now also R14.1
- net at Q2.2 (G), R16.2: now also R17.1
- net VCC renamed +5V
- net +5V: now also F3.1
- new net: Q3.2 (G), R19.2, R20.1
- new net: D2.2 (A), R15.2
- new net: D1.2 (A), R12.2
- new net: D3.2 (A), R18.2
- new net MOSFET_3: R18.1, R19.1
- new net SSR_3: Q3.1 (D)
- new net SSR_3_COM: F3.2
Other:
- moved on the sheet: F1, F2, Q1, Q2, R13, R14, R16, R17
