File: Hardware/Sheets/Microcontroller.kicad_sch (KiCad schematic)
At the start: 25 parts, among them IC1 MCP1792T, J9 POW_SEL, U1 W25Q16JV, U2 RP2040, Y1 12MHz

Commit message: minor work left on rev1
Parts:
- removed C13: 100n, KiCAD Library:C_0603_1608Metric, symbol Device:C_Small
- removed C16: 2u2, KiCAD Library:C_0603_1608Metric, symbol Device:C_Small
- removed IC1: MCP1792T, Package_TO_SOT_SMD:SOT-23, symbol SamacSys_Parts:MCP1792T-3302H_CB
- removed J9: POW_SEL, symbol Connector_Generic:Conn_01x03
- added C17: 2u2, KiCAD Library:C_0603_1608Metric, symbol Device:C_Small
- added J11: PawPad_SWD, PawPad:pawpad, symbol pawpad:PawPad_SWD
- added R2: DNF, Cuprum:R_0603_1608Metric, symbol Device:R_Small
- added SW1, SW2: DNF, KiCAD Library:PTS636 SM25J SMTR LFS, symbol Switch:SW_Push
- C15: value 10u -> 100n
Connections:
- net +1V1: no longer U2.23 (DVDD), U2.45 (VREG_VOUT), U2.50 (DVDD)
- net +3V3: now also C15.1, C17.1
- net GND: now also C17.2, J11.5 (GND), SW1.1, SW2.1
- net LED_ACTIVE: now also U2.37 (GPIO25); no longer U2.36 (GPIO24)
- net QSPI_SS: now also R2.1
- net SWCLK: now also J11.3 (SWCLK)
- net SWD: now also J11.2 (SWDIO)
- net ALARM1A: no longer names the net of U2.4 (GPIO2)
- net ALARM1B: no longer names the net of U2.8 (GPIO6)
- net ALARM2A: no longer names the net of U2.5 (GPIO3)
- net ALARM2B: no longer names the net of U2.9 (GPIO7)
- net ALARM3A: no longer names the net of U2.6 (GPIO4)
- net ALARM3B: no longer names the net of U2.11 (GPIO8)
- net ALARM4A: no longer names the net of U2.7 (GPIO5)
- net ALARM4B: no longer names the net of U2.12 (GPIO9)
- net ENC_A: no longer names the net of U2.14 (GPIO11)
- net ENC_B: no longer names the net of U2.15 (GPIO12)
- net ENC_SW: no longer names the net of U2.16 (GPIO13)
- net RUN renamed RST
- net RST: now also J11.4 (NRST), SW2.2
- net SW_EN: no longer names the net of U2.17 (GPIO14)
- net SW_LED: no longer names the net of U2.18 (GPIO15)
- new net: R2.2, SW1.2
- new net 1V1_B: U2.23 (DVDD), U2.45 (VREG_VOUT), U2.50 (DVDD)
- new net OUT_EN3: U2.36 (GPIO24)
- no-connect marks 7 -> 20
Other:
- note added: "BOOTSEL if needed"
- note added: "Programming"
- note added: "Reset"
- moved on the sheet: D2, R7
