File: Hardware/Sheets/USB.kicad_sch (KiCad schematic)
At the start: 4 parts, among them J5 USB4110-GF-A_REVB, U3 USBUF02W6

Commit message: minor work left on rev1
Parts:
- J11: renamed from J5; footprint KiCAD Library:GCT_USB4110-GF-A_REVB -> Connector_USB:USB_C_Receptacle_GCT_USB4105-xx-A_16P_TopMnt_Horizontal
- renumbered U3 to U1
Changed lines of the file:
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@@
+    (stroke (width 0) (type default))
+  )
+  (wire (pts (xy 109.22 91.44) (xy 116.84 91.44))
     (stroke (width 0) (type default))
   )
@@
   )
   (wire (pts (xy 138.43 95.25) (xy 109.22 95.25))
-    (stroke (width 0) (type default))
-  )
-  (wire (pts (xy 109.22 91.44) (xy 116.84 91.44))
     (stroke (width 0) (type default))
   )
@@
   (symbol (lib_id "power:+3V3") (at 175.26 99.06 0) (unit 1)
     (in_bom yes) (on_board yes) (dnp no) (fields_autoplaced)
-    (property "Reference" "#PWR041" (at 175.26 102.87 0)
+    (property "Reference" "#PWR025" (at 175.26 102.87 0)
       (effects (font (size 1.27 1.27)) hide)
     )
@@
       (project "Reflow Oven"
         (path "/a8f55c7f-bff8-431d-a8db-3e7e1d4b6c05/60f7cfdd-e831-4444-bc85-3a1c2ee14475"
-          (reference "#PWR041") (unit 1)
+          (reference "#PWR025") (unit 1)
         )
       )
@@
   (symbol (lib_id "power:VBUS") (at 116.84 85.09 0) (unit 1)
     (in_bom yes) (on_board yes) (dnp no) (fields_autoplaced)
-    (property "Reference" "#PWR039" (at 116.84 88.9 0)
+    (property "Reference" "#PWR023" (at 116.84 88.9 0)
       (effects (font (size 1.27 1.27)) hide)
     )
@@
       (project "Reflow Oven"
         (path "/a8f55c7f-bff8-431d-a8db-3e7e1d4b6c05/60f7cfdd-e831-4444-bc85-3a1c2ee14475"
-          (reference "#PWR039") (unit 1)
+          (reference "#PWR023") (unit 1)
         )
       )
@@
           (reference "R3") (unit 1)
         )
-        (path "/a8f55c7f-bff8-431d-a8db-3e7e1d4b6c05/c8b8f2ff-0b9b-4830-841d-05219ecaf535"
-          (reference "R1") (unit 1)
-        )
-        (path "/a8f55c7f-bff8-431d-a8db-3e7e1d4b6c05/60f7cfdd-e831-4444-bc85-3a1c2ee14475"
-          (reference "R15") (unit 1)
+        (path "/a8f55c7f-bff8-431d-a8db-3e7e1d4b6c05/60f7cfdd-e831-4444-bc85-3a1c2ee14475"
+          (reference "R10") (unit 1)
         )
       )
@@
   (symbol (lib_id "Connector:USB_C_Receptacle_USB2.0") (at 93.98 104.14 0) (unit 1)
     (in_bom yes) (on_board yes) (dnp no)
-    (property "Reference" "J5" (at 93.98 83.6635 0)
+    (property "Reference" "J11" (at 93.98 83.6635 0)
       (effects (font (size 1.27 1.27)))
     )
@@
       (effects (font (size 1.27 1.27)))
     )
-    (property "Footprint" "KiCAD Library:GCT_USB4110-GF-A_REVB" (at 97.79 104.14 0)
+    (property "Footprint" "Connector_USB:USB_C_Receptacle_GCT_USB4105-xx-A_16P_TopMnt_Horizontal" (at 97.79 104.14 0)
       (effects (font (size 1.27 1.27)) hide)
     )
@@
       (project "Reflow Oven"
         (path "/a8f55c7f-bff8-431d-a8db-3e7e1d4b6c05/60f7cfdd-e831-4444-bc85-3a1c2ee14475"
-          (reference "J5") (unit 1)
+          (reference "J11") (unit 1)
         )
       )
@@
           (reference "R3") (unit 1)
         )
-        (path "/a8f55c7f-bff8-431d-a8db-3e7e1d4b6c05/c8b8f2ff-0b9b-4830-841d-05219ecaf535"
-          (reference "R1") (unit 1)
-        )
-        (path "/a8f55c7f-bff8-431d-a8db-3e7e1d4b6c05/60f7cfdd-e831-4444-bc85-3a1c2ee14475"
-          (reference "R16") (unit 1)
+        (path "/a8f55c7f-bff8-431d-a8db-3e7e1d4b6c05/60f7cfdd-e831-4444-bc85-3a1c2ee14475"
+          (reference "R11") (unit 1)
         )
       )
@@
   (symbol (lib_id "Cuprum:USBUF02W6") (at 186.69 106.68 0) (unit 1)
     (in_bom yes) (on_board yes) (dnp no) (fields_autoplaced)
-    (property "Reference" "U3" (at 186.69 97.79 0)
+    (property "Reference" "U1" (at 186.69 97.79 0)
       (effects (font (size 1.27 1.27)))
     )
@@
       (project "Reflow Oven"
         (path "/a8f55c7f-bff8-431d-a8db-3e7e1d4b6c05/60f7cfdd-e831-4444-bc85-3a1c2ee14475"
-          (reference "U3") (unit 1)
+          (reference "U1") (unit 1)
         )
       )
@@
   (symbol (lib_id "power:GND") (at 86.36 134.62 0) (unit 1)
     (in_bom yes) (on_board yes) (dnp no) (fields_autoplaced)
-    (property "Reference" "#PWR038" (at 86.36 140.97 0)
+    (property "Reference" "#PWR022" (at 86.36 140.97 0)
       (effects (font (size 1.27 1.27)) hide)
     )
@@
       (project "Reflow Oven"
         (path "/a8f55c7f-bff8-431d-a8db-3e7e1d4b6c05/60f7cfdd-e831-4444-bc85-3a1c2ee14475"
-          (reference "#PWR038") (unit 1)
+          (reference "#PWR022") (unit 1)
         )
       )
@@
   (symbol (lib_id "PCM_4ms_Power-symbol:GND") (at 198.12 114.3 0) (unit 1)
     (in_bom yes) (on_board yes) (dnp no) (fields_autoplaced)
-    (property "Reference" "#PWR042" (at 198.12 120.65 0)
+    (property "Reference" "#PWR026" (at 198.12 120.65 0)
       (effects (font (size 1.27 1.27)) hide)
     )
@@
       (project "Reflow Oven"
         (path "/a8f55c7f-bff8-431d-a8db-3e7e1d4b6c05/60f7cfdd-e831-4444-bc85-3a1c2ee14475"
-          (reference "#PWR042") (unit 1)
+          (reference "#PWR026") (unit 1)
         )
       )
@@
   (symbol (lib_id "power:GND") (at 157.48 88.9 0) (unit 1)
     (in_bom yes) (on_board yes) (dnp no) (fields_autoplaced)
-    (property "Reference" "#PWR040" (at 157.48 95.25 0)
+    (property "Reference" "#PWR024" (at 157.48 95.25 0)
       (effects (font (size 1.27 1.27)) hide)
     )
@@
       (project "Reflow Oven"
         (path "/a8f55c7f-bff8-431d-a8db-3e7e1d4b6c05/60f7cfdd-e831-4444-bc85-3a1c2ee14475"
-          (reference "#PWR040") (unit 1)
-        )
-      )
+          (reference "#PWR024") (unit 1)
+        )
+      )

Commit message: minor tweaks
Connections:
- net GND: no longer J11.S1 (SHIELD), J11.S2 (SHIELD), J11.S3 (SHIELD), J11.S4 (SHIELD)
- no-connect marks 2 -> 6
Changed lines of the file:
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@@
   (junction (at 99.06 129.54) (diameter 0) (color 0 0 0 0)
   )
-  (junction (at 93.98 129.54) (diameter 0) (color 0 0 0 0)
-  )
-  (junction (at 86.36 129.54) (diameter 0) (color 0 0 0 0)
-  )
   (junction (at 111.76 109.22) (diameter 0) (color 0 0 0 0)
   )
-  (junction (at 88.9 129.54) (diameter 0) (color 0 0 0 0)
-  )
   (junction (at 111.76 104.14) (diameter 0) (color 0 0 0 0)
   )
-  (junction (at 91.44 129.54) (diameter 0) (color 0 0 0 0)
-  )
   (junction (at 147.32 85.09) (diameter 0) (color 0 0 0 0)
   )
   (junction (at 116.84 88.9) (diameter 0) (color 0 0 0 0)
   )
+  (no_connect (at 93.98 127))
+  (no_connect (at 88.9 127))
   (no_connect (at 109.22 113.03))
+  (no_connect (at 91.44 127))
   (no_connect (at 109.22 115.57))
+  (no_connect (at 86.36 127))
   (wire (pts (xy 157.48 85.09) (xy 157.48 88.9))
     (stroke (width 0) (type default))
@@
     (stroke (width 0) (type default))
   )
-  (wire (pts (xy 86.36 129.54) (xy 88.9 129.54))
-    (stroke (width 0) (type default))
-  )
   (wire (pts (xy 194.31 104.14) (xy 201.93 104.14))
     (stroke (width 0) (type default))
   )
-  (wire (pts (xy 99.06 129.54) (xy 93.98 129.54))
-    (stroke (width 0) (type default))
-  )
   (wire (pts (xy 198.12 106.68) (xy 194.31 106.68))
     (stroke (width 0) (type default))
   )
-  (wire (pts (xy 91.44 127) (xy 91.44 129.54))
+  (wire (pts (xy 99.06 132.08) (xy 99.06 129.54))
     (stroke (width 0) (type default))
   )
@@
     (stroke (width 0) (type default))
   )
-  (wire (pts (xy 88.9 129.54) (xy 91.44 129.54))
-    (stroke (width 0) (type default))
-  )
   (wire (pts (xy 101.6 127) (xy 101.6 129.54))
     (stroke (width 0) (type default))
@@
     (stroke (width 0) (type default))
   )
-  (wire (pts (xy 88.9 127) (xy 88.9 129.54))
-    (stroke (width 0) (type default))
-  )
-  (wire (pts (xy 91.44 129.54) (xy 93.98 129.54))
-    (stroke (width 0) (type default))
-  )
   (wire (pts (xy 109.22 104.14) (xy 111.76 104.14))
     (stroke (width 0) (type default))
@@
     (stroke (width 0) (type default))
   )
-  (wire (pts (xy 86.36 127) (xy 86.36 129.54))
-    (stroke (width 0) (type default))
-  )
   (wire (pts (xy 111.76 109.22) (xy 111.76 106.68))
     (stroke (width 0) (type default))
   )
   (wire (pts (xy 147.32 97.79) (xy 147.32 91.44))
-    (stroke (width 0) (type default))
-  )
-  (wire (pts (xy 93.98 127) (xy 93.98 129.54))
-    (stroke (width 0) (type default))
-  )
-  (wire (pts (xy 86.36 129.54) (xy 86.36 134.62))
     (stroke (width 0) (type default))
   )
@@
     )
   )
-  (symbol (lib_id "power:GND") (at 86.36 134.62 0) (unit 1)
-    (in_bom yes) (on_board yes) (dnp no) (fields_autoplaced)
-    (property "Reference" "#PWR022" (at 86.36 140.97 0)
-      (effects (font (size 1.27 1.27)) hide)
-    )
-    (property "Value" "GND" (at 86.36 139.1825 0)
-      (effects (font (size 1.27 1.27)))
-    )
-    (property "Footprint" "" (at 86.36 134.62 0)
-      (effects (font (size 1.27 1.27)) hide)
-    )
-    (property "Datasheet" "" (at 86.36 134.62 0)
-      (effects (font (size 1.27 1.27)) hide)
-    )
+  (symbol (lib_id "power:GND") (at 99.06 132.08 0) (unit 1)
+    (in_bom yes) (on_board yes) (dnp no) (fields_autoplaced)
+    (property "Reference" "#PWR022" (at 99.06 138.43 0)
+      (effects (font (size 1.27 1.27)) hide)
+    )
+    (property "Value" "GND" (at 99.06 136.6425 0)
+      (effects (font (size 1.27 1.27)))
+    )
+    (property "Footprint" "" (at 99.06 132.08 0)
+      (effects (font (size 1.27 1.27)) hide)
+    )
+    (property "Datasheet" "" (at 99.06 132.08 0)
+      (effects (font (size 1.27 1.27)) hide)
+    )
