File: Hardware/Rev 1/Reflow Oven.kicad_pcb (KiCad board)
At the start: 4 copper layers, 100 x 50 mm, 84 parts, among them IC1 MCP1792T, J1 SW, J10 2350513-2, J11 USB4110-GF-A_REVB, J12 POW_SEL, J13 PawPad_SWD, J2 ENC, J3 Adafruit 4101, J4 Adafruit 4101, J5 Adafruit 4101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

Commit message: functional prototype
Parts:
- added R27: 270, Cuprum:R_0603_1608Metric, F.Cu at (140.0, 84.8)
- J13: value PawPad_SWD -> Conn_01x02; footprint PawPad:pawpad -> Connector_PinHeader_2.54mm:PinHeader_1x02_P2.54mm_Vertical
- moved J13 0.88 mm to (140.0, 81.9), turned to 90 degrees
- moved R26 0.67 mm to (132.9, 81.8)
- moved D4 0.25 mm to (133.6, 79.0)
Connections:
- J13 pad 1: unconnected-(J13-SWO-Pad1) -> Net-(J13-Pin_1)
- J13 pad 2: /Microcontroller Alarm/SWD -> GND
- U4 pad 36: unconnected-(U4-GPIO24-Pad36) -> /Microcontroller Alarm/LED_FRONT
Routing:
- net /Microcontroller Alarm/LED_FRONT: track 0.00 -> 15.1 mm, vias 0 -> 2
- net /Microcontroller Alarm/SWCLK: track 11.2 -> 0.00 mm, vias 2 -> 0
- net /Microcontroller Alarm/SWD: track 9.83 -> 0.00 mm, vias 2 -> 0
- net /Microcontroller Alarm/RST: track 20.4 -> 16.7 mm
- net /ENC_Filter/ENC_SW_OUT: track 50.1 -> 47.5 mm
- net Net-(J13-Pin_1): track 0.00 -> 2.09 mm
- net /ENC_Filter/ENC_A_OUT: track 41.5 -> 43.2 mm
- net Net-(D4-A): track 1.69 -> 0.00 mm
- net GND: track 58.8 -> 57.2 mm, vias 38 -> 37
- net /SCL: track 86.8 -> 87.6 mm
- net /Microcontroller Alarm/LED_ACTIVE: track 1.96 -> 2.64 mm
- net /LCD_D/C: track 17.9 -> 17.3 mm
Other:
- board text added: "MCP9600 0x60"
- board text added: "MCP9600 0x61"
- board text added: "MCP9600 0x67"
- board text removed: "MCP9600"

Commit message: small pcb improvements
Routing:
- net /Microcontroller Alarm/USB_D-: track 16.1 -> 15.4 mm
- added copper zone on F.Cu, net Net-(D4-A)

Commit message: redid 2 layer, thanks git
Parts:
- moved J11 15.3 mm to (131.2, 57.3)
- moved C1 15.2 mm to (161.2, 79.5)
- moved C10 15.2 mm to (143.3, 73.2)
- moved C11 15.2 mm to (125.0, 83.8)
- moved C12 15.2 mm to (137.4, 81.8)
- moved C13 15.2 mm to (134.3, 66.8)
- moved C14 15.2 mm to (132.9, 66.8)
- moved C15 15.2 mm to (152.2, 78.8)
- moved C16 15.2 mm to (127.7, 75.0)
- moved C17 15.2 mm to (126.6, 75.0)
- moved C18 15.2 mm to (132.9, 79.2)
- moved C19 15.2 mm to (130.4, 70.2)
- moved C2 15.2 mm to (165.2, 79.5)
- moved C20 15.2 mm to (175.2, 81.6)
- moved C21 15.2 mm to (152.2, 73.8)
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Routing:
- net +3V3: track 45.3 -> 252.0 mm
- net GND: vias 37 -> 39
- added copper zone on B.Cu, net +3V3
- added copper zone on B.Cu, net GND
- removed copper zone on In1.Cu, net +3V3
- removed copper zone on In2.Cu, net GND
Other:
- copper layers 4 -> 2

Commit message: ordered from aisler
Parts:
- removed SW2: DNF, KiCAD Library:PTS636 SM25J SMTR LFS
Connections:
- U4 pad 26: /Microcontroller Alarm/RST -> unconnected-(U4-RUN-Pad26)
Routing:
- net /Microcontroller Alarm/RST: track 16.7 -> 0.00 mm
Other:
- board text added: "GC9A01 Display"
- board text added: "LED"
- board text added: "POW SEL"
- board text removed: "JLCJLCJLCJLC"
- board text removed: "LCD"
- board text removed: "Power Select"
- board text removed: "Reset"
Changed lines of the file:
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@@
   (net 38 "/Microcontroller Alarm/SWD")
   (net 39 "/Microcontroller Alarm/SWCLK")
-  (net 40 "/Microcontroller Alarm/RST")
+  (net 40 "unconnected-(U4-RUN-Pad26)")
   (net 41 "Net-(Q2-G)")
   (net 42 "Net-(Q3-G)")
@@
     )
   )
-  (footprint "KiCAD Library:PTS636 SM25J SMTR LFS" (layer "F.Cu")
-    (at 142.25 60)
-    (property "Sheetfile" "Sheets/MicrocontrollerAlarm.kicad_sch")
-    (property "Sheetname" "Microcontroller Alarm")
-    (property "ki_description" "Push button switch, generic, two pins")
-    (property "ki_keywords" "switch normally-open pushbutton push-button")
-    (attr smd)
-    (fp_text reference "SW2" (at 0 -0.75 unlocked) (layer "F.SilkS") hide
-        (effects (font (size 1 1) (thickness 0.15)))
-    )
-    (fp_text value "DNF" (at 0 1 unlocked) (layer "F.Fab")
-        (effects (font (size 1 1) (thickness 0.15)))
-    )
-    (fp_rect (start -4.4 -2.1) (end 4.4 2.1)
-      (stroke (width 0.1) (type solid)) (fill none) (layer "F.CrtYd"))
-    (fp_rect (start -3.05 -1.85) (end 3.05 1.85)
-      (stroke (width 0.1) (type solid)) (fill none) (layer "F.Fab"))
-    (fp_rect (start -1.35 -0.65) (end 1.35 0.65)
-      (stroke (width 0.1) (type solid)) (fill none) (layer "F.Fab"))
-    (pad "1" smd rect (at -3.775 0) (size 1.45 2.1) (layers "F.Cu" "F.Paste" "F.Mask")
-      (net 2 "GND") (pinfunction "1") (pintype "passive"))
-    (pad "2" smd rect (at 3.775 0) (size 1.45 2.1) (layers "F.Cu" "F.Paste" "F.Mask")
-      (net 40 "/Microcontroller Alarm/RST") (pinfunction "2") (pintype "passive"))
-    (model "${MODEL_3D}/PTS636SM25JSMTRLFS.step"
-      (offset (xyz 0 0 0))
-      (scale (xyz 1 1 1))
-      (rotate (xyz 0 0 0))
-    )
-  )
   (footprint "Connector_PinHeader_2.54mm:PinHeader_1x07_P2.54mm_Vertical" locked (layer "F.Cu")
     (at 153.12 56 -90)
@@
       (net 38 "/Microcontroller Alarm/SWD") (pinfunction "SWD") (pintype "bidirectional"))
     (pad "26" smd roundrect locked (at 1.8 3.4375 90) (size 0.2 0.875) (layers "F.Cu" "F.Paste" "F.Mask") (roundrect_rratio 0.25)
-      (net 40 "/Microcontroller Alarm/RST") (pinfunction "RUN") (pintype "input"))
+      (net 40 "unconnected-(U4-RUN-Pad26)") (pinfunction "RUN") (pintype "input+no_connect"))
     (pad "27" smd roundrect locked (at 2.2 3.4375 90) (size 0.2 0.875) (layers "F.Cu" "F.Paste" "F.Mask") (roundrect_rratio 0.25)
       (net 10 "/LCD_D{slash}C") (pinfunction "GPIO16") (pintype "bidirectional"))
@@
     (effects (font (size 1.5 1.5) (thickness 0.25) bold) (justify left bottom))
   )
+  (gr_text "LED" (at 142.534671 64.8) (layer "F.SilkS" knockout)
+    (effects (font (size 1 1) (thickness 0.15)) (justify left bottom))
+  )
   (gr_text "Button" (at 145.943928 82.9) (layer "F.SilkS" knockout)
     (effects (font (size 1 1) (thickness 0.15)) (justify left bottom))
   )
-  (gr_text "Power Select" (at 148.75 63.00869 -90) (layer "F.SilkS" knockout)
+  (gr_text "POW SEL" (at 148.75 64.603929 270) (layer "F.SilkS" knockout)
     (effects (font (size 1 1) (thickness 0.15)) (justify left bottom))
   )
@@
     (effects (font (size 1 1) (thickness 0.15)) (justify left bottom))
   )
-  (gr_text "JLCJLCJLCJLC" (at 158.65 58.275) (layer "F.SilkS")
-    (effects (font (size 1.5 1.5) (thickness 0.3) bold) (justify left bottom))
-  )
   (gr_text "SSR 1" (at 110.25 59.1) (layer "F.SilkS" knockout)
     (effects (font (size 1 1) (thickness 0.15)) (justify left bottom))
@@
     (effects (font (size 1.5 1.5) (thickness 0.25) bold) (justify left bottom))
   )
-  (gr_text "LCD" (at 149.1 59.65) (layer "F.SilkS" knockout)
+  (gr_text "GC9A01 Display" (at 139.564881 59.5) (layer "F.SilkS" knockout)
     (effects (font (size 1 1) (thickness 0.15)) (justify left bottom))
   )
@@
     (effects (font (size 1 1) (thickness 0.15)) (justify left bottom))
   )
-  (gr_text "Reset" (at 140.25 64) (layer "F.SilkS" knockout)
-    (effects (font (size 1 1) (thickness 0.15)) (justify left bottom))
-  )
   (gr_text "SSR 2" (at 110.25 71.2) (layer "F.SilkS" knockout)
     (effects (font (size 1 1) (thickness 0.15)) (justify left bottom))
@@
   (segment (start 122.4 91.025) (end 122.86 90.565) (width 0.2) (layer "F.Cu") (net 37))
   (segment (start 122.86 90.565) (end 122.86 88.192942) (width 0.2) (layer "F.Cu") (net 37))
-  (segment (start 140.9 64.8) (end 141.7 64) (width 0.2) (layer "F.Cu") (net 40))
-  (segment (start 140.302381 71.778991) (end 140.9 71.181372) (width 0.2) (layer "F.Cu") (net 40))
-  (segment (start 144.5 64) (end 146.025 62.475) (width 0.2) (layer "F.Cu") (net 40))
-  (segment (start 139.389324 71.778991) (end 140.302381 71.778991) (width 0.2) (layer "F.Cu") (net 40))
-  (segment (start 141.7 64) (end 144.5 64) (width 0.2) (layer "F.Cu") (net 40))
-  (segment (start 140.9 71.181372) (end 140.9 64.8) (width 0.2) (layer "F.Cu") (net 40))
-  (segment (start 146.025 62.475) (end 146.025 60) (width 0.2) (layer "F.Cu") (net 40))
   (segment (start 110.9125 62.2615) (end 116.2 62.2615) (width 0.25) (layer "F.Cu") (net 41))
   (segment (start 110.9125 74.3705) (end 116.2 74.3705) (width 0.25) (layer "F.Cu") (net 42))
