File: Hardware/Rev 1/Sheets/MicrocontrollerAlarm.kicad_sch (KiCad schematic)
At the start: 33 parts, among them IC1 MCP1792T, J13 PawPad_SWD, J9 POW_SEL, SW1 DNF, SW2 DNF, U1 W25Q16JV, U2 RP2040, U3 FT24C04A, Y1 12MHz

Commit message: functional prototype
Parts:
- removed J13: PawPad_SWD, PawPad:pawpad, symbol pawpad:PawPad_SWD
- added J13: Conn_01x02, Connector_PinHeader_2.54mm:PinHeader_1x02_P2.54mm_Vertical, symbol Connector_Generic:Conn_01x02
- added R7: 270, Cuprum:R_0603_1608Metric, symbol Device:R_Small
Connections:
- net GND: now also J13.2 (Pin_2)
- net LED_FRONT: now reaches U2.36 (GPIO24)
- net LED_FRONT: now also R7.2
- new net: J13.1 (Pin_1), R7.1
- no-connect marks 4 -> 2
Other:
- note removed: "PawPad"
Changed lines of the file:
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@@
   )
   (no_connect (at 181.61 137.16))
-  (no_connect (at 232.41 121.92))
-  (no_connect (at 149.86 176.53))
   (no_connect (at 232.41 137.16))
   (wire (pts (xy 125.73 165.1) (xy 111.76 165.1))
@@
     (stroke (width 0) (type default))
   )
-  (wire (pts (xy 142.24 179.07) (xy 149.86 179.07))
-    (stroke (width 0) (type default))
-  )
   (wire (pts (xy 27.94 127) (xy 40.64 127))
     (stroke (width 0) (type default))
@@
     (stroke (width 0) (type default))
   )
+  (wire (pts (xy 139.7 180.34) (xy 152.4 180.34))
+    (stroke (width 0) (type default))
+  )
   (wire (pts (xy 78.74 172.72) (xy 66.04 172.72))
     (stroke (width 0) (type default))
@@
     (stroke (width 0) (type default))
   )
+  (wire (pts (xy 156.21 182.88) (xy 160.02 182.88))
+    (stroke (width 0) (type default))
+  )
   (wire (pts (xy 68.58 85.09) (xy 58.42 85.09))
     (stroke (width 0) (type default))
@@
     (stroke (width 0) (type default))
   )
+  (wire (pts (xy 232.41 121.92) (xy 250.19 121.92))
+    (stroke (width 0) (type default))
+  )
   (wire (pts (xy 163.83 129.54) (xy 181.61 129.54))
     (stroke (width 0) (type default))
@@
     (stroke (width 0) (type default))
   )
+  (wire (pts (xy 156.21 182.88) (xy 156.21 185.42))
+    (stroke (width 0) (type default))
+  )
   (wire (pts (xy 62.23 30.48) (xy 62.23 33.02))
     (stroke (width 0) (type default))
@@
     (stroke (width 0) (type default))
   )
-  (wire (pts (xy 147.32 189.23) (xy 147.32 186.69))
-    (stroke (width 0) (type default))
-  )
   (wire (pts (xy 109.22 172.72) (xy 125.73 172.72))
     (stroke (width 0) (type default))
   )
-  (wire (pts (xy 147.32 186.69) (xy 149.86 186.69))
-    (stroke (width 0) (type default))
-  )
-  (wire (pts (xy 142.24 184.15) (xy 149.86 184.15))
-    (stroke (width 0) (type default))
-  )
   (wire (pts (xy 232.41 104.14) (xy 250.19 104.14))
     (stroke (width 0) (type default))
@@
     (stroke (width 0) (type default))
   )
-  (wire (pts (xy 142.24 181.61) (xy 149.86 181.61))
-    (stroke (width 0) (type default))
-  )
   (wire (pts (xy 49.53 119.38) (xy 49.53 124.46))
     (stroke (width 0) (type default))
@@
   )
   (wire (pts (xy 22.86 74.93) (xy 25.4 74.93))
+    (stroke (width 0) (type default))
+  )
+  (wire (pts (xy 157.48 180.34) (xy 160.02 180.34))
     (stroke (width 0) (type default))
   )
@@
     (effects (font (size 2 2)) (justify left bottom))
   )
-  (text "PawPad" (at 138.43 170.18 0)
-    (effects (font (size 2 2)) (justify left bottom))
-  )
   (text "Oscillator" (at 16.51 59.69 0)
     (effects (font (size 2 2)) (justify left bottom))
@@
     (effects (font (size 1.27 1.27)) (justify right bottom))
   )
-  (label "RST" (at 142.24 184.15 0) (fields_autoplaced)
-    (effects (font (size 1.27 1.27)) (justify left bottom))
-  )
   (label "QSPI_SD0" (at 78.74 167.64 180) (fields_autoplaced)
     (effects (font (size 1.27 1.27)) (justify right bottom))
@@
     (effects (font (size 1.27 1.27)) (justify right bottom))
   )
+  (label "LED_FRONT" (at 139.7 180.34 0) (fields_autoplaced)
+    (effects (font (size 1.27 1.27)) (justify left bottom))
+  )
   (label "QSPI_SD2" (at 78.74 172.72 180) (fields_autoplaced)
     (effects (font (size 1.27 1.27)) (justify right bottom))
@@
     (effects (font (size 1.27 1.27)) (justify left bottom))
   )
+  (label "LED_FRONT" (at 250.19 121.92 180) (fields_autoplaced)
+    (effects (font (size 1.27 1.27)) (justify right bottom))
+  )
   (label "QSPI_SS" (at 163.83 78.74 0) (fields_autoplaced)
     (effects (font (size 1.27 1.27)) (justify left bottom))
@@
   (label "SCL" (at 67.31 124.46 180) (fields_autoplaced)
     (effects (font (size 1.27 1.27)) (justify right bottom))
-  )
-  (label "SWD" (at 142.24 179.07 0) (fields_autoplaced)
-    (effects (font (size 1.27 1.27)) (justify left bottom))
-  )
-  (label "SWCLK" (at 142.24 181.61 0) (fields_autoplaced)
-    (effects (font (size 1.27 1.27)) (justify left bottom))
   )
   (label "LED_ACTIVE" (at 78.74 71.12 0) (fields_autoplaced)
@@
         (path "/dbd87a35-3166-440e-a8f0-c71d214a12a6/5b814077-791b-4a8a-adc0-955088325477"
           (reference "#PWR038") (unit 1)
+        )
+      )
+    )
+  )
+  (symbol (lib_id "Device:R_Small") (at 154.94 180.34 270) (unit 1)
+    (in_bom yes) (on_board yes) (dnp no) (fields_autoplaced)
+    (property "Reference" "R7" (at 154.94 175.26 90)
+      (effects (font (size 1.27 1.27)))
+    )
+    (property "Value" "270" (at 154.94 177.8 90)
+      (effects (font (size 1.27 1.27)))
+    )
+    (property "Footprint" "Cuprum:R_0603_1608Metric" (at 154.94 180.34 0)
+      (effects (font (size 1.27 1.27)) hide)
+    )
+    (property "Datasheet" "~" (at 154.94 180.34 0)
+      (effects (font (size 1.27 1.27)) hide)
+    )
+    (pin "1")
+    (pin "2")
+    (instances
+      (project "Reflow Oven"
+        (path "/a8f55c7f-bff8-431d-a8db-3e7e1d4b6c05"
+          (reference "R7") (unit 1)
+        )
+        (path "/a8f55c7f-bff8-431d-a8db-3e7e1d4b6c05/43b08574-0fed-4e0b-a6ee-f48c75075e2f"
+          (reference "R27") (unit 1)
+        )
+      )
+      (project "USB-PD"
+        (path "/dbd87a35-3166-440e-a8f0-c71d214a12a6"
+          (reference "R?") (unit 1)
+        )
+        (path "/dbd87a35-3166-440e-a8f0-c71d214a12a6/0250254d-69b0-47eb-8561-149d95a16e02"
+          (reference "R9") (unit 1)
+        )
+        (path "/dbd87a35-3166-440e-a8f0-c71d214a12a6/ba296704-8a9e-4bdd-ada8-fe9cd67794b5"
+          (reference "R12") (unit 1)
+        )
+        (path "/dbd87a35-3166-440e-a8f0-c71d214a12a6/e00e204b-d6fc-451e-8397-028d03c22f27"
+          (reference "R14") (unit 1)
         )
       )
@@
     )
   )
-  (symbol (lib_id "pawpad:PawPad_SWD") (at 156.21 181.61 0) (unit 1)
-    (in_bom yes) (on_board yes) (dnp no) (fields_autoplaced)
-    (property "Reference" "J13" (at 161.29 180.6575 0)
-      (effects (font (size 1.27 1.27)) (justify left))
-    )
-    (property "Value" "PawPad_SWD" (at 161.29 183.1975 0)
-      (effects (font (size 1.27 1.27)) (justify left))
-    )
-    (property "Footprint" "PawPad:pawpad" (at 156.21 193.675 0)
-      (effects (font (size 1.27 1.27)) hide)
-    )
-    (property "Datasheet" "" (at 153.67 178.435 0)
-      (effects (font (size 1.27 1.27)) hide)
-    )
-    (pin "1")
-    (pin "2")
-    (pin "3")
-    (pin "4")
-    (pin "5")
+  (symbol (lib_id "Connector_Generic:Conn_01x02") (at 165.1 180.34 0) (unit 1)
+    (in_bom yes) (on_board yes) (dnp no)
+    (property "Reference" "J13" (at 163.83 177.8 0)
+      (effects (font (size 1.27 1.27)) (justify left))
+    )
+    (property "Value" "Conn_01x02" (at 160.02 185.42 0)
+      (effects (font (size 1.27 1.27)) (justify left))
+    )
+    (property "Footprint" "Connector_PinHeader_2.54mm:PinHeader_1x02_P2.54mm_Vertical" (at 165.1 180.34 0)
+      (effects (font (size 1.27 1.27)) hide)
+    )
+    (property "Datasheet" "~" (at 165.1 180.34 0)
+      (effects (font (size 1.27 1.27)) hide)
+    )
+    (pin "1")
+    (pin "2")
     (instances
       (project "Reflow Oven"
@@
         (path "/dbd87a35-3166-440e-a8f0-c71d214a12a6/5b814077-791b-4a8a-adc0-955088325477"
           (reference "C20") (unit 1)
-        )
-      )
-    )
-  )
-  (symbol (lib_id "power:GND") (at 147.32 189.23 0) (unit 1)
-    (in_bom yes) (on_board yes) (dnp no)
-    (property "Reference" "#PWR017" (at 147.32 195.58 0)
-      (effects (font (size 1.27 1.27)) hide)
-    )
-    (property "Value" "GND" (at 147.447 193.6242 0)
-      (effects (font (size 1.27 1.27)))
-    )
-    (property "Footprint" "" (at 147.32 189.23 0)
-      (effects (font (size 1.27 1.27)) hide)
-    )
-    (property "Datasheet" "" (at 147.32 189.23 0)
-      (effects (font (size 1.27 1.27)) hide)
-    )
-    (pin "1")
-    (instances
-      (project "Reflow Oven"
-        (path "/a8f55c7f-bff8-431d-a8db-3e7e1d4b6c05"
-          (reference "#PWR017") (unit 1)
-        )
-        (path "/a8f55c7f-bff8-431d-a8db-3e7e1d4b6c05/43b08574-0fed-4e0b-a6ee-f48c75075e2f"
-          (reference "#PWR053") (unit 1)
-        )
-      )
-      (project "USB-PD"
-        (path "/dbd87a35-3166-440e-a8f0-c71d214a12a6"
-          (reference "#PWR?") (unit 1)
-        )
-        (path "/dbd87a35-3166-440e-a8f0-c71d214a12a6/5b814077-791b-4a8a-adc0-955088325477"
-          (reference "#PWR039") (unit 1)
         )
       )
@@
         )
       )
+    )
+  )
+  (symbol (lib_id "power:GND") (at 156.21 185.42 0) (unit 1)
+    (in_bom yes) (on_board yes) (dnp no) (fields_autoplaced)
+    (property "Reference" "#PWR031" (at 156.21 191.77 0)
+      (effects (font (size 1.27 1.27)) hide)
+    )
+    (property "Value" "GND" (at 156.21 189.9825 0)
+      (effects (font (size 1.27 1.27)))
+    )
+    (property "Footprint" "" (at 156.21 185.42 0)
+      (effects (font (size 1.27 1.27)) hide)
+    )
+    (property "Datasheet" "" (at 156.21 185.42 0)
+      (effects (font (size 1.27 1.27)) hide)
+    )
+    (pin "1")
+    (instances
+      (project "Reflow Oven"
+        (path "/a8f55c7f-bff8-431d-a8db-3e7e1d4b6c05/43b08574-0fed-4e0b-a6ee-f48c75075e2f"
+          (reference "#PWR031") (unit 1)
+        )
+      )
+      (project "USB-PD"
+        (path "/dbd87a35-3166-440e-a8f0-c71d214a12a6"
+          (reference "#PWR?") (unit 1)
+        )
+        (path "/dbd87a35-3166-440e-a8f0-c71d214a12a6/0250254d-69b0-47eb-8561-149d95a16e02"
+          (reference "#PWR014") (unit 1)
+        )
+      )

Commit message: ordered from aisler
Parts:
- removed SW2: DNF, KiCAD Library:PTS636 SM25J SMTR LFS, symbol Switch:SW_Push
Connections:
- net RST: no longer names the net of U2.26 (RUN)
- no-connect marks 2 -> 3
Changed lines of the file:
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@@
   )
   (no_connect (at 181.61 137.16))
+  (no_connect (at 181.61 60.96))
   (no_connect (at 232.41 137.16))
   (wire (pts (xy 125.73 165.1) (xy 111.76 165.1))
@@
     (stroke (width 0) (type default))
   )
-  (wire (pts (xy 142.24 62.23) (xy 142.24 60.96))
-    (stroke (width 0) (type default))
-  )
   (wire (pts (xy 232.41 91.44) (xy 250.19 91.44))
     (stroke (width 0) (type default))
@@
     (stroke (width 0) (type default))
   )
-  (wire (pts (xy 142.24 60.96) (xy 147.32 60.96))
-    (stroke (width 0) (type default))
-  )
   (wire (pts (xy 62.23 30.48) (xy 71.12 30.48))
     (stroke (width 0) (type default))
@@
   )
   (wire (pts (xy 232.41 60.96) (xy 250.19 60.96))
-    (stroke (width 0) (type default))
-  )
-  (wire (pts (xy 157.48 60.96) (xy 181.61 60.96))
     (stroke (width 0) (type default))
   )
@@
   (label "QSPI_SD0" (at 78.74 167.64 180) (fields_autoplaced)
     (effects (font (size 1.27 1.27)) (justify right bottom))
-  )
-  (label "RST" (at 163.83 60.96 0) (fields_autoplaced)
-    (effects (font (size 1.27 1.27)) (justify left bottom))
   )
   (label "SDA" (at 250.19 60.96 180) (fields_autoplaced)
@@
         (path "/dbd87a35-3166-440e-a8f0-c71d214a12a6/e00e204b-d6fc-451e-8397-028d03c22f27"
           (reference "R14") (unit 1)
-        )
-      )
-    )
-  )
-  (symbol (lib_id "power:GND") (at 142.24 62.23 0) (unit 1)
-    (in_bom yes) (on_board yes) (dnp no) (fields_autoplaced)
-    (property "Reference" "#PWR012" (at 142.24 68.58 0)
-      (effects (font (size 1.27 1.27)) hide)
-    )
-    (property "Value" "GND" (at 142.24 66.7925 0)
-      (effects (font (size 1.27 1.27)))
-    )
-    (property "Footprint" "" (at 142.24 62.23 0)
-      (effects (font (size 1.27 1.27)) hide)
-    )
-    (property "Datasheet" "" (at 142.24 62.23 0)
-      (effects (font (size 1.27 1.27)) hide)
-    )
-    (pin "1")
-    (instances
-      (project "Reflow Oven"
-        (path "/a8f55c7f-bff8-431d-a8db-3e7e1d4b6c05"
-          (reference "#PWR012") (unit 1)
-        )
-        (path "/a8f55c7f-bff8-431d-a8db-3e7e1d4b6c05/43b08574-0fed-4e0b-a6ee-f48c75075e2f"
-          (reference "#PWR052") (unit 1)
-        )
-      )
-      (project "USB-PD"
-        (path "/dbd87a35-3166-440e-a8f0-c71d214a12a6"
-          (reference "#PWR?") (unit 1)
-        )
-        (path "/dbd87a35-3166-440e-a8f0-c71d214a12a6/e00e204b-d6fc-451e-8397-028d03c22f27"
-          (reference "#PWR051") (unit 1)
         )
       )
@@
         )
       )
-    )
-  )
-  (symbol (lib_id "Switch:SW_Push") (at 152.4 60.96 0) (unit 1)
-    (in_bom yes) (on_board yes) (dnp no)
-    (property "Reference" "SW2" (at 152.4 55.88 0)
-      (effects (font (size 1.27 1.27)))
-    )
-    (property "Value" "DNF" (at 152.4 55.88 0)
-      (effects (font (size 1.27 1.27)) hide)
-    )
-    (property "Footprint" "KiCAD Library:PTS636 SM25J SMTR LFS" (at 152.4 55.88 0)
-      (effects (font (size 1.27 1.27)) hide)
-    )
-    (property "Datasheet" "~" (at 152.4 55.88 0)
-      (effects (font (size 1.27 1.27)) hide)
-    )
-    (pin "1")
-    (pin "2")
-    (instances
-      (project "Reflow Oven"
-        (path "/a8f55c7f-bff8-431d-a8db-3e7e1d4b6c05/43b08574-0fed-4e0b-a6ee-f48c75075e2f"
-          (reference "SW2") (unit 1)
-        )
-      )
-      (project "USB-PD"
-        (path "/dbd87a35-3166-440e-a8f0-c71d214a12a6"
-          (reference "SW?") (unit 1)
-        )
-        (path "/dbd87a35-3166-440e-a8f0-c71d214a12a6/6306dd5a-5b79-432e-ad73-0295989b9f81"
-          (reference "SW3") (unit 1)
-        )
-        (path "/dbd87a35-3166-440e-a8f0-c71d214a12a6/e00e204b-d6fc-451e-8397-028d03c22f27"
-          (reference "SW4") (unit 1)
-        )
-      )

Commit message: updated the schematic with the value for R21
Other:
- note added: "R21 should be between 1-10k R22 should not be fitted"
Changed lines of the file:
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@@
     (effects (font (size 2 2)) (justify left bottom))
+  )
+  (text "R21 should be between 1-10k\nR22 should not be fitted\n"
+    (at 19.05 144.78 0)
+    (effects (font (size 1.27 1.27)) (justify left bottom))
   )
   (text "Make sure C19 is close to pin 44" (at 96.52 45.72 0)
